Commit message: urdf/tiago_pro.urdf
Set all grippers joints to fixed

File: capsules/urdf/tiago_pro_capsules.urdf (robot description, URDF)
Before this commit: robot tiago_pro, 74 links, 73 joints
Joints:
- joint gripper_left_finger_joint: type prismatic -> fixed
- joint gripper_left_finger_right_joint: type prismatic -> fixed
- joint gripper_left_fingertip_left_joint: type revolute -> fixed
- joint gripper_left_fingertip_right_joint: type revolute -> fixed
- joint gripper_left_inner_finger_left_joint: type revolute -> fixed
- joint gripper_left_inner_finger_right_joint: type revolute -> fixed
- joint gripper_left_outer_finger_left_joint: type revolute -> fixed
- joint gripper_left_outer_finger_right_joint: type revolute -> fixed
- joint gripper_right_finger_joint: type prismatic -> fixed
- joint gripper_right_finger_right_joint: type prismatic -> fixed
- joint gripper_right_fingertip_left_joint: type revolute -> fixed
- joint gripper_right_fingertip_right_joint: type revolute -> fixed
- joint gripper_right_inner_finger_left_joint: type revolute -> fixed
- joint gripper_right_inner_finger_right_joint: type revolute -> fixed
- joint gripper_right_outer_finger_left_joint: type revolute -> fixed
- joint gripper_right_outer_finger_right_joint: type revolute -> fixed
