Commit message: telepresence_experiments

File: capsules/urdf/tiago_dual_capsules.urdf (robot description, URDF)
Before this commit: robot tiago_dual, 60 links, 59 joints
Links:
- link gripper_right_left_finger_link: geometry collision cylinder length=0.1268779539832169 radius=0.3268195; visual mesh filename=package://pal_gripper_description/meshes/gripper_finger_lin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

Commit message: rename capsules .rviz to urdf, keep only nice capsules instead of cylinders as collision urdf

File: capsules/urdf/tiago_dual_capsules.urdf (robot description, URDF)
Before this commit: robot tiago_dual, 60 links, 59 joints
Links:
- added link camera_head_frame
- added link camera_left_frame
- added link camera_right_frame
- added link world
- link arm_left_1_link: geometry collision cylinder length=0.12825732419899807 radius=0.0623321; collision sphere radius=0.0623321
- link arm_left_2_link: geometry collision cylinder length=0.0462256735826997 radius=0.0615206; collision sphere radius=0.0615206
- link arm_left_3_link: geometry collision cylinder length=0.18430979587454732 radius=0.0685082; collision sphere radius=0.0685082
- link arm_left_4_link: geometry collision cylinder length=0.07893204272296257 radius=0.0679987; collision sphere radius=0.0679987
- link arm_left_5_link: geometry collision cylinder length=0.10935921148420999 radius=0.0685869; collision sphere radius=0.0685869
- link arm_left_6_link: geometry collision cylinder length=0.033837367068951754 radius=0.04237; collision sphere radius=0.04237
- link arm_left_tool_link: geometry collision cylinder length=0.005 radius=0.005; collision sphere radius=0.005
- link arm_right_1_link: geometry collision cylinder length=0.12825732419899807 radius=0.0623321; collision sphere radius=0.0623321
- link arm_right_2_link: geometry collision cylinder length=0.0462256735826997 radius=0.0615206; collision sphere radius=0.0615206
- link arm_right_3_link: geometry collision cylinder length=0.18430979587454732 radius=0.0685082; collision sphere radius=0.0685082
- link arm_right_4_link: geometry collision cylinder length=0.07892139663102109 radius=0.0680003; collision sphere radius=0.0680003
- link arm_right_5_link: geometry collision cylinder length=0.1091053809489577 radius=0.068611; collision sphere radius=0.068611
- link arm_right_6_link: geometry collision cylinder length=0.033837367068951754 radius=0.04237; collision sphere radius=0.04237
- link arm_right_tool_link: geometry collision cylinder length=0.005 radius=0.005; collision sphere radius=0.005
- link base_antenna_left_link: geometry collision cylinder length=0.12302074541933909 radius=0.0295745; collision sphere radius=0.0295745
- link base_antenna_right_link: geometry collision cylinder length=0.12302074541933909 radius=0.0295745; collision sphere radius=0.0295745
- link base_dock_link: geometry collision cylinder length=0.0419972 radius=0.0293112; collision sphere radius=0.0293112
- link base_front_laser_link: geometry 
- link base_link: geometry collision cylinder length=0.392504 radius=0.26807; collision sphere radius=0.26807
- link base_rear_laser_link: geometry 
- link gripper_left_left_finger_link: geometry collision cylinder length=0.1268779539832169 radius=0.0268195; collision sphere radius=0.0268195
- link gripper_left_link: geometry collision cylinder length=0.05239620003790586 radius=0.0651301; collision sphere radius=0.0651301
- link gripper_left_right_finger_link: geometry collision cylinder length=0.12361389657269042 radius=0.0266004; collision sphere radius=0.0266004
- link gripper_right_left_finger_link: geometry collision cylinder length=0.1268779539832169 radius=0.0268195; collision sphere radius=0.0268195
- link gripper_right_link: geometry collision cylinder length=0.05239620003790586 radius=0.0651301; collision sphere radius=0.0651301
- link gripper_right_right_finger_link: geometry collision cylinder length=0.12361389657269042 radius=0.0266004; collision sphere radius=0.0266004
- link head_1_link: geometry collision cylinder length=0.03803007097377325 radius=0.087289; collision sphere radius=0.087289
- link head_2_link: geometry collision cylinder length=0.12273180000004075 radius=0.118353; collision sphere radius=0.118353
- link suspension_front_left_link: geometry collision cylinder length=0.10696387374307084 radius=0.0403258; collision sphere radius=0.0403258
- link suspension_front_right_link: geometry collision cylinder length=0.10696387374307084 radius=0.0403258; collision sphere radius=0.0403258
- link suspension_rear_left_link: geometry collision cylinder length=0.10616482685182932 radius=0.0403527; collision sphere radius=0.0403527
- link suspension_rear_right_link: geometry collision cylinder length=0.10616482685182932 radius=0.0403527; collision sphere radius=0.0403527
- link torso_fixed_link: geometry collision cylinder length=0.27767100694629604 radius=0.139555; collision sphere radius=0.139555
- link torso_lift_link: geometry collision cylinder length=0.27845962332116486 radius=0.22228; collision sphere radius=0.22228
- link wheel_front_left_link: geometry collision cylinder length=0.05 radius=0.0762; collision sphere radius=0.0762
- link wheel_front_right_link: geometry collision cylinder length=0.05 radius=0.0762; collision sphere radius=0.0762
- link wheel_rear_left_link: geometry collision cylinder length=0.05 radius=0.0762; collision sphere radius=0.0762
- link wheel_rear_right_link: geometry collision cylinder length=0.05 radius=0.0762; collision sphere radius=0.0762
- link wrist_left_ft_link: geometry collision cylinder length=0.0157 radius=0.0225; collision sphere radius=0.0225
- link wrist_left_ft_tool_link: geometry collision cylinder length=0.00975 radius=0.025; collision sphere radius=0.025
- link wrist_right_ft_link: geometry collision cylinder length=0.0157 radius=0.0225; collision sphere radius=0.0225
- link wrist_right_ft_tool_link: geometry collision cylinder length=0.00975 radius=0.025; collision sphere radius=0.025
Joints:
- added joint camera_head_frame_joint: type fixed, parent base_link, child camera_head_frame, origin xyz=0.171591 0.0112369 1.20358 rpy=-3.1415927 0.0 0.0
- added joint camera_left_frame_joint: type fixed, parent wrist_left_ft_tool_link, child camera_left_frame, origin xyz=0.072 -0.085 -0.032 rpy=1.57079632679 0 0
- added joint camera_right_frame_joint: type fixed, parent wrist_right_ft_tool_link, child camera_right_frame, origin xyz=0.072 -0.085 -0.032 rpy=1.57079632679 0 0
- added joint reference: type floating, parent world, child base_footprint

File: capsules/urdf/tiago_pro_capsules.urdf (robot description, URDF)
Before this commit: robot tiago_pro, 74 links, 73 joints
Links:
- link arm_left_1_link: geometry collision cylinder length=0.14549002180106163 radius=0.05485; collision sphere radius=0.05485
- link arm_left_2_link: geometry collision cylinder length=0.14226556572150903 radius=0.0487698; collision sphere radius=0.0487698
- link arm_left_3_link: geometry collision cylinder length=0.14549002187610613 radius=0.05485; collision sphere radius=0.05485
- link arm_left_4_link: geometry collision cylinder length=0.14226556572150903 radius=0.0487698; collision sphere radius=0.0487698
- link arm_left_5_link: geometry collision cylinder length=0.16908291531885833 radius=0.0445055; collision sphere radius=0.0445055
- link arm_left_6_link: geometry collision cylinder length=0.05419845669846048 radius=0.0648013; collision sphere radius=0.0648013
- link arm_left_7_link: geometry collision cylinder length=0.006640813932186702 radius=0.0427711; collision sphere radius=0.0427711
- link arm_right_1_link: geometry collision cylinder length=0.14549002180106163 radius=0.05485; collision sphere radius=0.05485
- link arm_right_2_link: geometry collision cylinder length=0.14226556572150903 radius=0.0487698; collision sphere radius=0.0487698
- link arm_right_3_link: geometry collision cylinder length=0.14549002187610613 radius=0.05485; collision sphere radius=0.05485
- link arm_right_4_link: geometry collision cylinder length=0.14226556572150903 radius=0.0487698; collision sphere radius=0.0487698
- link arm_right_5_link: geometry collision cylinder length=0.16908291531885833 radius=0.0445055; collision sphere radius=0.0445055
- link arm_right_6_link: geometry collision cylinder length=0.05419845669846048 radius=0.0648013; collision sphere radius=0.0648013
- link arm_right_7_link: geometry collision cylinder length=0.006640813932186702 radius=0.0427711; collision sphere radius=0.0427711
- link base_antenna_left_link: geometry collision cylinder length=0.12302074541933909 radius=0.0295745; collision sphere radius=0.0295745
- link base_antenna_right_link: geometry collision cylinder length=0.12302074541933909 radius=0.0295745; collision sphere radius=0.0295745
- link base_dock_link: geometry collision cylinder length=0.0419972 radius=0.0293112; collision sphere radius=0.0293112
- link base_front_laser_link: geometry collision cylinder length=0.01 radius=0.01; collision sphere radius=0.01
- link base_link: geometry collision cylinder length=0.3920240000012837 radius=0.268189; collision sphere radius=0.268189
- link base_rear_laser_link: geometry collision cylinder length=0.01 radius=0.01; collision sphere radius=0.01
- link gripper_left_base_link: geometry collision cylinder length=0.0696281123961164 radius=0.038333; collision sphere radius=0.038333
- link gripper_left_fingertip_left_link: geometry collision cylinder length=0.036830457634388934 radius=0.0179351; collision sphere radius=0.0179351
- link gripper_left_fingertip_right_link: geometry collision cylinder length=0.036830457634388934 radius=0.0179351; collision sphere radius=0.0179351
- link gripper_left_inner_finger_left_link: geometry collision cylinder length=0.04259153403066128 radius=0.019791; collision sphere radius=0.019791
- link gripper_left_inner_finger_right_link: geometry collision cylinder length=0.04259153403066128 radius=0.019791; collision sphere radius=0.019791
- link gripper_left_outer_finger_left_link: geometry collision cylinder length=0.059493192471946406 radius=0.013095; collision sphere radius=0.013095
- link gripper_left_outer_finger_right_link: geometry collision cylinder length=0.059493192471946406 radius=0.013095; collision sphere radius=0.013095
- link gripper_right_base_link: geometry collision cylinder length=0.0696281123961164 radius=0.038333; collision sphere radius=0.038333
- link gripper_right_fingertip_left_link: geometry collision cylinder length=0.036830457634388934 radius=0.0179351; collision sphere radius=0.0179351
- link gripper_right_fingertip_right_link: geometry collision cylinder length=0.036830457634388934 radius=0.0179351; collision sphere radius=0.0179351
- link gripper_right_inner_finger_left_link: geometry collision cylinder length=0.04259153403066128 radius=0.019791; collision sphere radius=0.019791
- link gripper_right_inner_finger_right_link: geometry collision cylinder length=0.04259153403066128 radius=0.019791; collision sphere radius=0.019791
- link gripper_right_outer_finger_left_link: geometry collision cylinder length=0.059493192471946406 radius=0.013095; collision sphere radius=0.013095
- link gripper_right_outer_finger_right_link: geometry collision cylinder length=0.059493192471946406 radius=0.013095; collision sphere radius=0.013095
- link head_1_link: geometry collision cylinder length=0.045626321699621684 radius=0.0737178; collision sphere radius=0.0737178
- link head_2_link: geometry collision cylinder length=0.09910494482986204 radius=0.141531; collision sphere radius=0.141531
- link laptop_tray: geometry collision cylinder length=0.16198730615100554 radius=0.120001; collision sphere radius=0.120001
- link suspension_front_left_link: geometry collision cylinder length=0.10616482685182932 radius=0.0403527; collision sphere radius=0.0403527
- link suspension_front_right_link: geometry collision cylinder length=0.10616482685182932 radius=0.0403527; collision sphere radius=0.0403527
- link suspension_rear_left_link: geometry collision cylinder length=0.10616482685182932 radius=0.0403527; collision sphere radius=0.0403527
- link suspension_rear_right_link: geometry collision cylinder length=0.10616482685182932 radius=0.0403527; collision sphere radius=0.0403527
- link torso_base_link: geometry collision cylinder length=0.32749980143345386 radius=0.222419; collision sphere radius=0.222419
- link torso_lift_link: geometry collision cylinder length=0.09891795716337973 radius=0.23528; collision sphere radius=0.23528
- link wheel_front_left_link: geometry collision cylinder length=0.05 radius=0.0762; collision sphere radius=0.0762
- link wheel_front_right_link: geometry collision cylinder length=0.05 radius=0.0762; collision sphere radius=0.0762
- link wheel_rear_left_link: geometry collision cylinder length=0.05 radius=0.0762; collision sphere radius=0.0762
- link wheel_rear_right_link: geometry collision cylinder length=0.05 radius=0.0762; collision sphere radius=0.0762
